File: hardware/Kicad project/SWN v1.1/SWN.sch (KiCad schematic (older format))
At the start: 39 parts, among them J3 Conn_02x04_Odd_Even, U7 STM32F765ZG, U8 S25FL127, X1 16MHz

Commit message: Schematic symbol library alias created for F765 chip
Symbol changed to F765 in schematic
Parts:
- U7: symbol SMR-eagle:STM32F429ZI -> SMR-eagle:STM32F765ZG
Changed lines of the file:
@@
 $EndComp
 $Comp
-L SMR-eagle:STM32F429ZI U7
+L SMR-eagle:STM32F765ZG U7
 U 1 1 5935E939
 P 5375 4675
