File: hardware/Kicad project/SWN v1.1/swn-audio.sch (KiCad schematic (older format))
At the start: 40 parts, among them IC5 NJM2068, IC7 MCP1703x-3302E/MB, U1 WM8731, U24 TLV171

Commit message: Schematic updated to use KiCad 5.1.4 and new 4ms-vreg library.
Parts:
- IC7: symbol 4ms-ic:MCP1703x-XX02E -> 4ms-vreg:MCP1703x-XX02E
Changed lines of the file:
@@
 EESchema Schematic File Version 4
 LIBS:SWN-cache
-EELAYER 29 0
+EELAYER 30 0
 EELAYER END
 $Descr B 17000 11000
@@
 $EndComp
 $Comp
-L 4ms-ic:MCP1703x-XX02E IC?
+L 4ms-vreg:MCP1703x-XX02E IC?
 U 1 1 59BB4DD6
 P 4150 6450
