File: hardware/Kicad project/SWN v1.1/swn-power.sch (KiCad schematic (older format))
At the start: 23 parts, among them IC10 LD1117ADT33TR, J1 HEADER-1X3-TH, J2 HEADER-2X8-TH, U23 MCP1703x-3302E/MB

Commit message: Schematic updated to use KiCad 5.1.4 and new 4ms-vreg library.
Parts:
- IC10: symbol 4ms-ic:LD1117ADT -> 4ms-vreg:LD1117ADT
- U23: symbol 4ms-ic:MCP1703x-XX02E -> 4ms-vreg:MCP1703x-XX02E
Changed lines of the file:
@@
 EESchema Schematic File Version 4
 LIBS:SWN-cache
-EELAYER 29 0
+EELAYER 30 0
 EELAYER END
 $Descr B 17000 11000
@@
 $EndComp
 $Comp
-L 4ms-ic:LD1117ADT IC10
+L 4ms-vreg:LD1117ADT IC10
 U 1 1 593794F5
 P 7550 3975
@@
 $EndComp
 $Comp
-L 4ms-ic:MCP1703x-XX02E U23
+L 4ms-vreg:MCP1703x-XX02E U23
 U 1 1 59BC1766
 P 10850 2650
