File: hardware/Kicad project/SWN v1.1/swn-voctadc.sch (KiCad schematic (older format))
At the start: 101 parts, among them IC8 TL082, U14 TLV171, U15 ADS8634, U16 TLV171, U17 ADS8634, U18 TLV171, U19 TLV171, U20 TLV171, U21 TLV171

Commit message: Schematic updated to use KiCad 5.1.4 and new 4ms-vreg library.
Parts:
- V1: symbol 4ms-ic:KA78L05 -> 4ms-vreg:KA78L05
- V2: symbol 4ms-ic:ADR_VREF -> 4ms-vreg:ADR_VREF
Changed lines of the file:
@@
 EESchema Schematic File Version 4
 LIBS:SWN-cache
-EELAYER 29 0
+EELAYER 30 0
 EELAYER END
 $Descr B 17000 11000
@@
 $EndComp
 $Comp
-L 4ms-ic:KA78L05 V?
+L 4ms-vreg:KA78L05 V?
 U 1 1 59B9CC96
 P 8550 9150
@@
 	7850 9100 7250 9100
 $Comp
-L 4ms-ic:ADR_VREF V2
+L 4ms-vreg:ADR_VREF V2
 U 1 1 5B35F5EF
 P 4350 7900
+AR Path="/5B35F5EF" Ref="V2"  Part="1"
+AR Path="/59AF0AB3/5B35F5EF" Ref="V2"  Part="1"
 F 0 "V2" H 4125 8225 70  0000 L BNN
 F 1 "ADR381ARTZ" H 4100 8125 70  0000 L BNN
